Commit message: Updated Readme and Refactoring

File: safemotions/description/urdf/robot_ball_machine.urdf (robot description, URDF)
Before this commit: robot main, 10 links, 9 joints
Links:
- added link ball_machine, mass 1.0; collision mesh filename=package://safemotions/description/meshes/misc/collision/bal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 scale=2.2 2.2 2.2; visual mesh filename=package://safemotions/description/meshes/misc/visual/ball_m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 scale=2.2 2.2 2.2
- added link basketball, mass .0; visual mesh filename=package://safemotions/description/meshes/obstacles/visual/b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 scale=0.001076 0.001076 0.001076
Joints:
- added joint ball_machine_joint: type fixed, parent iiwa_link_7, child ball_machine, origin xyz=0 0.175 0.1645 rpy=1.570796 0 0
- added joint basketball_joint: type fixed, parent ball_machine, child basketball, origin xyz=0.0009 0.001 0.25 rpy=0 0 1.5707
